File: p3/main.sch (KiCad schematic (older format))
At the start: 15 parts, among them IC1 ATTINY45-P, P1 CONN_XT60, P2 CONN_01X06, P3 CONN_01X02, P4 CONN_XT60, Q1 BSS138, U1 AUIPS7111S, U2 LM3480-5.0, U3 74LVC1G08

Commit message: test
Parts:
- removed IC1: ATTINY45-P, Housings_SOIC:SOIC-8_3.9x4.9mm_Pitch1.27mm, symbol ATTINY45-P
- removed P1, P4: CONN_XT60, KiCad-MDH-Connectors:XT60, symbol CONN_XT60
- removed P3: CONN_01X02, Connectors_Hirose:Hirose_DF13C-02P-1.25V_02x1.25mm_Straight, symbol CONN_01X02
- added D? (x2): LED, symbol LED
- added IC1: ATTINY84-S, Housings_SOIC:SOIC-14_3.9x8.7mm_Pitch1.27mm, symbol ATTINY84-S
- added P1, P4, P5, P6: CONN_01X01, Mounting_Holes:MountingHole_3.2mm_M3_Pad_Via, symbol CONN_01X01
- added P3: CONN_01X03, Connectors_Hirose:Hirose_DF13-03P-1.25DS_03x1.25mm_Angled, symbol CONN_01X03
- added P7: CONN_01X02, Connectors_Hirose:Hirose_DF13-02P-1.25DS_02x1.25mm_Angled, symbol CONN_01X02
- added U? (x2): NSI45020AT1G, symbol NSI45020AT1G
- P2: footprint Connectors_Hirose:Hirose_DF13C-06P-1.25V_06x1.25mm_Straight -> Connectors_Hirose:Hirose_DF13-06P-1.25DS_06x1.25mm_Angled
Connections:
- net ENB1: now also IC1.10 ((PCINT3/T0/ADC3)PA3)
- net ENB2: now also P3.3 (P3)
- net GND: now also P2.6 (P6), D?.1 (K), D?.1 (K), IC1.14 (GND), P3.1 (P1), P4.1 (P1), P6.1 (P1), P7.1 (P1); no longer P2.1 (P1)
- net Ifb: now also R3.2; no longer R3.1
- net MISO: now also P2.3 (P3), IC1.8 ((PCINT5/DO/MISO/OC1B/ADC5)PA5); no longer P2.4 (P4)
- net Out: now also P5.1 (P1)
- net RESET: now also IC1.4 ((PCINT11/dW/~RESET~)PB3)
- net SCL/SCK: now also P2.4 (P4), IC1.9 ((PCINT4/USCK/SCL/T1/ADC4)PA4); no longer P2.5 (P5)
- net SDA/MOSI: now also P2.1 (P1), IC1.7 ((PCINT6/SDA/DI/MOSI/OC1A/ADC6)PA6); no longer P2.3 (P3)
- net VCC: now also P1.1 (P1)
- net +3V3 renamed +5V
- net +5V: now also P2.5 (P5), IC1.1 (VCC), P3.2 (P2); no longer P2.6 (P6)
- new net: D?.2 (A), U?.1 (x2)
- new net Current_Feedback: IC1.12 ((PCINT1/AIN0/ADC1)PA1), R3.1
- new net LED2: IC1.11 ((PCINT2/AIN1/ADC2)PA2)
- new net LED3: IC1.13 ((PCINT0/AREF/ADC0)PA0)
- new net PWM1: IC1.5 ((PCINT10/CKOUT/OC0A/INT0)PB2), P7.2 (P2)
- new net PWM2: IC1.6 ((PCINT7/ICP/OC0B/ADC7)PA7)
Other:
- moved on the sheet: C3, C4, P2, Q1, R1, R2, R3, R4, U1, U2, U3
